File: Morpho.kicad_sch (KiCad schematic)
At the start: 1 part, among them U4 NUCLEO-G474RE

Commit message: Generated scaffold for mcu2 finished brake sense rev2 finished adding second chip to nucleo devboard
Connections:
- net +3.3V renamed +3V3
Changed lines of the file:
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@@
 			)
 		)
-		(property "Value" "+3.3V"
+		(property "Value" "+3V3"
 			(at 131.318 72.39 90)
 			(show_name no)
