File: usb.kicad_sch (KiCad schematic)
At the start: 16 parts, among them J1 USB_B_Micro, U3 CP2102C-Axx-xQFN24

Commit message: Added finishing thouches to brake sense pcb Finished main schematic layout and added chosen component footprints Placed components in layout and started tracing
Parts:
- removed C7: 22u, Capacitor_SMD:C_0805_2012Metric, symbol Device:C
- removed D1: PTVS5VP, Diode_SMD:Nexperia_DSN1608-2_1.6x0.8mm, symbol Diode:PTVS5V0Z1USKP
- removed D3: ESD5.0V, Diode_SMD:D_SOD-923, symbol Diode:ESD9B5.0ST5G
- removed J1: USB_B_Micro, Connector_USB:USB_Micro-B_Amphenol_10103594-0001LF_Horizontal, symbol Connector:USB_B_Micro
- added D1: PTVS5V, Diode_SMD:D_SOD-123, symbol Diode:PTVS5V0Z1USK
- added J6: USB4105-GF-A, tinynav:USB4105_GCT, symbol tinynav:USB4105-GF-A
- added R14, R15: 5.1k, Resistor_SMD:R_0603_1608Metric, symbol Device:R
- added U2: USBLC6-2SC6, Package_TO_SOT_SMD:SOT-23-6, symbol Power_Protection:USBLC6-2SC6
- C5: renamed from C10; value 0.1uF -> 100nF; footprint Capacitor_SMD:C_0805_2012Metric -> Capacitor_SMD:C_0603_1608Metric
- C7: renamed from C12; value 0.1uF -> 100nF; footprint Capacitor_SMD:C_0805_2012Metric -> Capacitor_SMD:C_0603_1608Metric
- FB1: footprint Inductor_SMD:L_Panasonic_PCC-M0540M -> Inductor_SMD:L_0805_2012Metric
- R1: renamed from R8; footprint Resistor_SMD:R_0805_2012Metric -> Resistor_SMD:R_0603_1608Metric
- R2: renamed from R7; footprint Resistor_SMD:R_0805_2012Metric -> Resistor_SMD:R_0603_1608Metric
- renumbered C9 to C4, C11 to C6, R6 to R3, R9 to R4
Connections:
- net GND: now also D1.2 (A), J6.A1-B12 (GND), J6.B1-A12 (GND), R14.2, R15.1, U2.2 (GND)
- net USB_D_N: now also U2.4 (I/O2)
- net USB_D_P: now also U2.6 (I/O1)
- net VBUS: now also D1.1 (K), J6.A4-B9 (VBUS), J6.B4-A9 (VBUS), U2.5 (VBUS)
- new net: J6.A5 (CC1), R15.2
- new net: J6.B5 (CC2), R14.1
- new net DN: J6.A7 (DN1), J6.B7 (DN2), U2.3 (I/O2)
- new net DP: J6.A6 (DP1), J6.B6 (DP2), U2.1 (I/O1)
Other:
- moved on the sheet: C1, C2, C4, C5, C6, C7, FB1, R1, R2, R3, R4, U3

Commit message: added rev04_mcu1/2.h revised brake sense board Added logic for 2 MCUs on nucleo board
Other:
- moved on the sheet: U2

Commit message: Generated scaffold for mcu2 finished brake sense rev2 finished adding second chip to nucleo devboard
Changed lines of the file:
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@@
+	(wire
+		(pts
+			(xy 53.34 81.915) (xy 53.34 83.82)
+		)
+		(stroke
+			(width 0)
+			(type default)
+		)
+	)
 	(wire
 		(pts
@@
 					(unit 1)
 				)
+			)
+		)
+	)
+	(symbol
+		(lib_id "power:PWR_FLAG")
+		(at 53.34 81.915 0)
+		(unit 1)
+		(body_style 1)
+		(exclude_from_sim no)
+		(in_bom yes)
+		(on_board yes)
+		(in_pos_files yes)
+		(dnp no)
+		(fields_autoplaced yes)
+		(property "Reference" "#FLG06"
+			(at 53.34 80.01 0)
+			(hide yes)
+			(show_name no)
+			(do_not_autoplace no)
+			(effects
+				(font
+					(size 1.27 1.27)
+				)
+			)
+		)
+		(property "Value" "PWR_FLAG"
+			(at 53.34 76.835 0)
+			(show_name no)
+			(do_not_autoplace no)
+			(effects
+				(font
+					(size 1.27 1.27)
+				)
+			)
+		)
+		(property "Footprint" ""
+			(at 53.34 81.915 0)
+			(hide yes)
+			(show_name no)
+			(do_not_autoplace no)
+			(effects
+				(font
+					(size 1.27 1.27)
+				)
+			)
+		)
+		(property "Datasheet" ""
+			(at 53.34 81.915 0)
+			(hide yes)
+			(show_name no)
+			(do_not_autoplace no)
+			(effects
+				(font
+					(size 1.27 1.27)
+				)
+			)
+		)
+		(property "Description" "Special symbol for telling ERC where power comes from"
+			(at 53.34 81.915 0)
+			(hide yes)
+			(show_name no)
+			(do_not_autoplace no)
+			(effects
+				(font
+					(size 1.27 1.27)
+				)
+			)
+		)
+		(pin "1"
+		)
+		(instances
+			(project "Nucleo_devboard"
+				(path "/4250c3cc-f8c5-441a-9e80-e89bb6ada756/0682989f-1baf-459e-b0ed-fe1064436fe6"
+					(reference "#FLG06")
+					(unit 1)
+				)
