File: Nucleo_devboard.kicad_pcb (KiCad board)
At the start: 4 copper layers, 70 x 82.5 mm, 90 parts, among them J1 st_debug_SMD, J2 st_debug_SMD, J3 USB_5V, J4 E5V, J5 Curr_measure, J6 USB4105-GF-A, J7 Conn_01x03_Socket, J8 CAN, U1 STM32G474RETx, U2 USBLC6-2SC6, U3 CP2102C-Axx-xQFN24, U4 NUCLEO-G474RE, U5 TLV75533PDBV, U6 STM32G474RETx, U7 MCP2562-E-SN, Y1 Crystal 24MHz, Y2 Crystal 32.768KHz, Y3 Crystal 24MHz

Commit message: Commit before reference renaming
Parts:
- added D9: D_Dual_CommonCathode_AAK_Parallel, Package_TO_SOT_SMD:SOT-23, F.Cu at (1.96, 1.73)
- C12, C14: value 1μF -> 1uF
- moved C28 1.80 mm to (144.6, 120.8)
- moved C27 1.80 mm to (144.6, 122.6)
- moved C43 1.49 mm to (133.7, 142.0), turned to 180 degrees
Routing:
- net GND: track 127.9 -> 129.5 mm
- net +3V3: track 67.3 -> 66.6 mm
