File: Power_sel.kicad_sch (KiCad schematic)
At the start: 13 parts, among them J3 USB_5V, J4 E5V, J5 Curr_measure, U5 TLV75533PDBV

Commit message: Generated scaffold for mcu2 finished brake sense rev2 finished adding second chip to nucleo devboard
Parts:
- D5, D6: value BAT60JFILM -> BAT60A
Changed lines of the file:
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@@
 			)
 		)
-		(property "Value" "BAT60JFILM"
+		(property "Value" "BAT60A"
 			(at 109.22 73.6599 90)
 			(show_name no)
@@
 			)
 		)
-		(property "Value" "BAT60JFILM"
+		(property "Value" "BAT60A"
 			(at 91.44 73.6599 90)
 			(show_name no)

Commit message: Finished last thouches on brake sense and nucleo pcb (Ordered pcbs)
Parts:
- renumbered D5 to D2, D6 to D3, D2 to D5
Changed lines of the file:
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@@
 		(dnp no)
 		(fields_autoplaced yes)
-		(property "Reference" "D6"
+		(property "Reference" "D3"
 			(at 109.22 71.1199 90)
 			(show_name no)
@@
 			(project "Nucleo_devboard"
 				(path "/4250c3cc-f8c5-441a-9e80-e89bb6ada756/b44e4b98-b890-48d2-b758-cee07234a0bd"
-					(reference "D6")
+					(reference "D3")
 					(unit 1)
 				)
@@
 		(dnp no)
 		(fields_autoplaced yes)
-		(property "Reference" "D5"
+		(property "Reference" "D2"
 			(at 91.44 71.1199 90)
 			(show_name no)
@@
 			(project "Nucleo_devboard"
 				(path "/4250c3cc-f8c5-441a-9e80-e89bb6ada756/b44e4b98-b890-48d2-b758-cee07234a0bd"
-					(reference "D5")
+					(reference "D2")
 					(unit 1)
 				)
@@
 		(in_pos_files yes)
 		(dnp no)
-		(property "Reference" "D2"
+		(property "Reference" "D5"
 			(at 202.692 60.452 0)
 			(show_name no)
@@
 			(project "Nucleo_devboard"
 				(path "/4250c3cc-f8c5-441a-9e80-e89bb6ada756/b44e4b98-b890-48d2-b758-cee07234a0bd"
-					(reference "D2")
-					(unit 1)
-				)
+					(reference "D5")
+					(unit 1)
+				)

Commit message: volvo_h2 revision Revised switch regulator layout/components Changed brake circuit to use current sense amplifier Defined nets and nettclass constraints. Revises trace layout to fit new constraints.
Parts:
- J3, J4, J5: footprint tinynav:HARWIN_M20-9990246 -> tinynav:jumper_header; symbol tinynav:M20-9990246 -> tinynav:jumper_header
Changed lines of the file:
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@@
 	)
 	(symbol
-		(lib_id "tinynav:M20-9990246")
+		(lib_id "tinynav:jumper_header")
 		(at 86.36 85.09 270)
 		(unit 1)
@@
 			)
 		)
-		(property "Footprint" "tinynav:HARWIN_M20-9990246"
+		(property "Footprint" "tinynav:jumper_header"
 			(at 86.36 85.09 0)
 			(hide yes)
@@
 	)
 	(symbol
-		(lib_id "tinynav:M20-9990246")
+		(lib_id "tinynav:jumper_header")
 		(at 104.14 85.09 270)
 		(unit 1)
@@
 			)
 		)
-		(property "Footprint" "tinynav:HARWIN_M20-9990246"
+		(property "Footprint" "tinynav:jumper_header"
 			(at 104.14 85.09 0)
 			(hide yes)
@@
 	)
 	(symbol
-		(lib_id "tinynav:M20-9990246")
+		(lib_id "tinynav:jumper_header")
 		(at 181.61 73.66 270)
 		(unit 1)
@@
 			)
 		)
-		(property "Footprint" "tinynav:HARWIN_M20-9990246"
+		(property "Footprint" "tinynav:jumper_header"
 			(at 181.61 73.66 0)
 			(hide yes)

Commit message: Commit before reference renaming
Parts:
- added D9: D_Dual_CommonCathode_AAK_Parallel, Package_TO_SOT_SMD:SOT-23, symbol Device:D_Dual_CommonCathode_AAK_Parallel
- C12, C14: value 1μF -> 1uF
Changed lines of the file:
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@@
 			)
 		)
-		(property "Value" "1μF"
+		(property "Value" "1uF"
 			(at 132.842 77.216 0)
 			(show_name no)
@@
 	)
 	(symbol
+		(lib_id "Device:D_Dual_CommonCathode_AAK_Parallel")
+		(at 128.27 43.815 0)
+		(unit 1)
+		(body_style 1)
+		(exclude_from_sim no)
+		(in_bom yes)
+		(on_board yes)
+		(in_pos_files yes)
+		(dnp no)
+		(fields_autoplaced yes)
+		(property "Reference" "D9"
+			(at 128.2065 35.56 0)
+			(show_name no)
+			(do_not_autoplace no)
+			(effects
+				(font
+					(size 1.27 1.27)
+				)
+			)
+		)
+		(property "Value" "D_Dual_CommonCathode_AAK_Parallel"
+			(at 128.2065 38.1 0)
+			(show_name no)
+			(do_not_autoplace no)
+			(effects
+				(font
+					(size 1.27 1.27)
+				)
+			)
+		)
+		(property "Footprint" "Package_TO_SOT_SMD:SOT-23"
+			(at 129.54 43.815 0)
+			(hide yes)
+			(show_name no)
+			(do_not_autoplace no)
+			(effects
+				(font
+					(size 1.27 1.27)
+				)
+			)
+		)
+		(property "Datasheet" ""
+			(at 129.54 43.815 0)
+			(hide yes)
+			(show_name no)
+			(do_not_autoplace no)
+			(effects
+				(font
+					(size 1.27 1.27)
+				)
+			)
+		)
+		(property "Description" "Dual diode, common cathode on pin 1"
+			(at 128.27 43.815 0)
+			(hide yes)
+			(show_name no)
+			(do_not_autoplace no)
+			(effects
+				(font
+					(size 1.27 1.27)
+				)
+			)
+		)
+		(pin "1"
+		)
+		(pin "3"
+		)
+		(pin "2"
+		)
+		(instances
+			(project "Nucleo_devboard"
+				(path "/4250c3cc-f8c5-441a-9e80-e89bb6ada756/b44e4b98-b890-48d2-b758-cee07234a0bd"
+					(reference "D9")
+					(unit 1)
+				)
+			)
+		)
+	)
+	(symbol
 		(lib_id "Device:D_Zener")
 		(at 88.9 72.39 270)
@@
 			)
 		)
-		(property "Value" "1μF"
+		(property "Value" "1uF"
 			(at 168.656 77.47 0)
 			(show_name no)
